File: hardware/FV-CTRL_RevA2.kicad_pcb (KiCad board)
At the start: 2 copper layers, 100 x 100 mm, 76 parts, among them J1 12V INPUT, J10 IR RX2 3V3/OUT/G, J11 IR TX1 A/K, J12 IR TX2 A/K, J13 LS1 DNP, J14 LS2 DNP, J15 LS3 DNP, J16 LS4 DNP, J17 I2C 3V3/SDA/SCL/G, J18 DEVKITC V4 LEFT, J19 DEVKITC V4 RIGHT, J2 XL4015 A: 12/G/6/G, J3 XL4015 B: 12/G/6/G, J4 5V D24V25F5, J5 S1_TOP, J6 S1_BOT, J7 S2_TOP, J8 S2_BOT, J9 IR RX1 3V3/OUT/G, Q1 IRF4905PBF, Q2 P2N2222AG

Commit message: Add external IR pullups and qualify RevA2 component sourcing
Parts:
- added R26: 10k, Resistor_THT:R_Axial_DIN0207_L6.3mm_D2.5mm_P7.62mm_Horizontal, F.Cu at (129.0, 135.0)
- added R27: 10k, Resistor_THT:R_Axial_DIN0207_L6.3mm_D2.5mm_P7.62mm_Horizontal, F.Cu at (122.0, 155.0)
- added R28: 1k, Resistor_THT:R_Axial_DIN0207_L6.3mm_D2.5mm_P7.62mm_Horizontal, F.Cu at (126.0, 155.0)
- added R29: 1k, Resistor_THT:R_Axial_DIN0207_L6.3mm_D2.5mm_P7.62mm_Horizontal, F.Cu at (126.0, 165.0)
- C5: value 10uF 25V -> 10uF 50V
- TP1, TP2, TP3, TP4, TP5, TP6, TP7, TP8: footprint TestPoint:TestPoint_THTPad_D3.0mm_Drill1.5mm -> fv_reva2:Keystone_5000_Carrier_D3
- moved C9 61.4 mm to (133.0, 135.0), turned to 90 degrees
- moved TP8 37.5 mm to (161.0, 179.0)
- moved D5 29.8 mm to (129.0, 124.0), turned to 90 degrees
- moved C7 21.9 mm to (109.0, 119.0), turned to 0 degrees
- moved C6 18.6 mm to (122.0, 118.0)
- moved D2 16.4 mm to (118.0, 119.0), turned to 90 degrees
- moved D6 15.0 mm to (123.0, 184.0), turned to -90 degrees
- moved TP4 11.0 mm to (131.0, 117.0)
- moved C10 8.94 mm to (113.0, 193.0), turned to -90 degrees
- moved C8 6.32 mm to (136.0, 129.0), turned to 0 degrees
- moved TP6 2.00 mm to (126.0, 114.0)
Connections:
- J10 pad 2: /IR_RX2 -> /IR_RX2_CABLE
- J9 pad 2: /IR_RX1 -> /IR_RX1_CABLE
Routing:
- net /GND: track 14.1 -> 505.3 mm
- net /+12V: track 111.4 -> 140.3 mm
- net /LED5_A: track 6.75 -> 34.8 mm, vias 0 -> 1
- net /LED2_A: track 18.4 -> 45.4 mm, vias 0 -> 1
- net /IR_RX2_CABLE: track 0.00 -> 22.4 mm
- net /IR_RX1_CABLE: track 0.00 -> 21.5 mm
- net /+5V: track 137.8 -> 116.8 mm, vias 0 -> 1
- net /LED6_A: track 14.4 -> 33.6 mm, vias 0 -> 2
- net /SPARE_GPIO33: track 21.4 -> 36.7 mm, vias 0 -> 1
- net /I2C_SCL: track 66.4 -> 56.2 mm
- net /S2_TOP_PWM: track 19.0 -> 28.6 mm
- net /LS1: track 104.4 -> 113.2 mm, vias 0 -> 2
- net /LS4: track 125.5 -> 119.2 mm
- net /LS3: track 116.3 -> 121.6 mm, vias 0 -> 1
- net /IR_TX2_A: track 42.4 -> 47.7 mm
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