File: hardware/FV-CTRL_RevA2.kicad_sch (KiCad schematic)
At the start: 72 parts, among them J1 12V INPUT, J10 IR RX2 3V3/OUT/G, J11 IR TX1 A/K, J12 IR TX2 A/K, J13 LS1 DNP, J14 LS2 DNP, J15 LS3 DNP, J16 LS4 DNP, J17 I2C 3V3/SDA/SCL/G, J18 DEVKITC V4 LEFT, J19 DEVKITC V4 RIGHT, J2 XL4015 A: 12/G/6/G, J3 XL4015 B: 12/G/6/G, J4 5V D24V25F5, J5 S1_TOP, J6 S1_BOT, J7 S2_TOP, J8 S2_BOT, J9 IR RX1 3V3/OUT/G, Q1 IRF4905PBF, Q2 P2N2222AG

Commit message: feat(pcb): route RevA2 with 2mm power paths and clean parity DRC
Parts:
- added H1, H2, H3, H4: M3 MOUNT, MountingHole:MountingHole_3.2mm_M3, symbol Mechanical:MountingHole
Connections:
- net +12V: now also J4.2 (Pin_2); no longer J4.4 (Pin_4)
- net +5V: now also J4.5 (Pin_5); no longer J4.1 (Pin_1)
- net GND: now also J4.4 (Pin_4); no longer J4.2 (Pin_2)
Other:
- note added: "LIMIT DNP / MOUNTING"
- note removed: "LIMIT DNP"
Changed lines of the file:
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@@
 		(fill (type none))
 	)
-	(text "LIMIT DNP"
+	(text "LIMIT DNP / MOUNTING"
 		(exclude_from_sim no)
 		(at 538.7200 20.0800 0)
@@
 	)
 	(symbol
+		(lib_id "Mechanical:MountingHole")
+		(at 585.4700 355.6000 0)
+		(unit 1)
+		(exclude_from_sim no)
+		(in_bom yes)
+		(on_board yes)
+		(dnp no)
+		(property "Reference" "H1"
+			(at 585.4700 353.0600 0)
+			(effects (font (size 1.27 1.27)))
+		)
+		(property "Value" "M3 MOUNT"
+			(at 585.4700 358.1400 0)
+			(effects (font (size 1.27 1.27)))
+		)
+		(property "Footprint" "MountingHole:MountingHole_3.2mm_M3"
+			(at 585.4700 355.6000 0)
+			(effects (font (size 1.27 1.27)) (hide yes))
+		)
+		(property "Datasheet" "~"
+			(at 585.4700 355.6000 0)
+			(effects (font (size 1.27 1.27)) (hide yes))
+		)
+		(property "Description" ""
+			(at 585.4700 355.6000 0)
+			(effects (font (size 1.27 1.27)) (hide yes))
+		)
+		(pin "1")
+		(pin "2")
+	)
+	(symbol
+		(lib_id "Mechanical:MountingHole")
+		(at 585.4700 382.2700 0)
+		(unit 1)
+		(exclude_from_sim no)
+		(in_bom yes)
+		(on_board yes)
+		(dnp no)
+		(property "Reference" "H2"
+			(at 585.4700 379.7300 0)
+			(effects (font (size 1.27 1.27)))
+		)
+		(property "Value" "M3 MOUNT"
+			(at 585.4700 384.8100 0)
+			(effects (font (size 1.27 1.27)))
+		)
+		(property "Footprint" "MountingHole:MountingHole_3.2mm_M3"
+			(at 585.4700 382.2700 0)
+			(effects (font (size 1.27 1.27)) (hide yes))
+		)
+		(property "Datasheet" "~"
+			(at 585.4700 382.2700 0)
+			(effects (font (size 1.27 1.27)) (hide yes))
+		)
+		(property "Description" ""
+			(at 585.4700 382.2700 0)
+			(effects (font (size 1.27 1.27)) (hide yes))
+		)
+		(pin "1")
+		(pin "2")
+	)
+	(symbol
+		(lib_id "Mechanical:MountingHole")
+		(at 585.4700 408.9400 0)
+		(unit 1)
+		(exclude_from_sim no)
+		(in_bom yes)
+		(on_board yes)
+		(dnp no)
+		(property "Reference" "H3"
+			(at 585.4700 406.4000 0)
+			(effects (font (size 1.27 1.27)))
+		)
+		(property "Value" "M3 MOUNT"
+			(at 585.4700 411.4800 0)
+			(effects (font (size 1.27 1.27)))
+		)
+		(property "Footprint" "MountingHole:MountingHole_3.2mm_M3"
+			(at 585.4700 408.9400 0)
+			(effects (font (size 1.27 1.27)) (hide yes))
+		)
+		(property "Datasheet" "~"
+			(at 585.4700 408.9400 0)
+			(effects (font (size 1.27 1.27)) (hide yes))
+		)
+		(property "Description" ""
+			(at 585.4700 408.9400 0)
+			(effects (font (size 1.27 1.27)) (hide yes))
+		)
+		(pin "1")
+		(pin "2")
+	)
+	(symbol
+		(lib_id "Mechanical:MountingHole")
+		(at 585.4700 435.6100 0)
+		(unit 1)
+		(exclude_from_sim no)
+		(in_bom yes)
+		(on_board yes)
+		(dnp no)
+		(property "Reference" "H4"
+			(at 585.4700 433.0700 0)
+			(effects (font (size 1.27 1.27)))
+		)
+		(property "Value" "M3 MOUNT"
+			(at 585.4700 438.1500 0)
+			(effects (font (size 1.27 1.27)))
+		)
+		(property "Footprint" "MountingHole:MountingHole_3.2mm_M3"
+			(at 585.4700 435.6100 0)
+			(effects (font (size 1.27 1.27)) (hide yes))
+		)
+		(property "Datasheet" "~"
+			(at 585.4700 435.6100 0)
+			(effects (font (size 1.27 1.27)) (hide yes))
+		)
+		(property "Description" ""
+			(at 585.4700 435.6100 0)
+			(effects (font (size 1.27 1.27)) (hide yes))
+		)
+		(pin "1")
+		(pin "2")
+	)
+	(symbol
 		(lib_id "Device:R")
 		(at 715.0100 35.5600 0)
@@
 	(wire
 		(pts
-			(xy 60.9600 403.8600) (xy 55.8800 403.8600)
+			(xy 60.9600 406.4000) (xy 55.8800 406.4000)
 		)
 		(stroke (width 0) (type default))
@@
 	(wire
 		(pts
-			(xy 60.9600 406.4000) (xy 55.8800 406.4000)
+			(xy 60.9600 408.9400) (xy 55.8800 408.9400)
 		)
 		(stroke (width 0) (type default))
@@
 	(wire
 		(pts
-			(xy 60.9600 408.9400) (xy 55.8800 408.9400)
+			(xy 60.9600 411.4800) (xy 55.8800 411.4800)
 		)
 		(stroke (width 0) (type default))
@@
 	(wire
 		(pts
-			(xy 60.9600 411.4800) (xy 55.8800 411.4800)
+			(xy 60.9600 414.0200) (xy 55.8800 414.0200)
 		)
 		(stroke (width 0) (type default))
@@
 		(effects (font (size 1.27 1.27)))
 	)
-	(label "+5V"
-		(at 55.8800 403.8600 0)
-		(effects (font (size 1.27 1.27)))
-	)
-	(label "GND"
+	(label "+12V"
 		(at 55.8800 406.4000 0)
 		(effects (font (size 1.27 1.27)))
@@
 		(effects (font (size 1.27 1.27)))
 	)
-	(label "+12V"
+	(label "GND"
 		(at 55.8800 411.4800 0)
 		(effects (font (size 1.27 1.27)))
 	)
 	(label "+5V"
+		(at 55.8800 414.0200 0)
+		(effects (font (size 1.27 1.27)))
+	)
+	(label "+5V"
 		(at 55.8800 436.8800 0)
 		(effects (font (size 1.27 1.27)))
@@
 	)
 	(no_connect
-		(at 60.9600 414.0200)
+		(at 60.9600 403.8600)
 	)
 	(no_connect

Commit message: Add external IR pullups and qualify RevA2 component sourcing
Parts:
- added R26, R27: 10k, Resistor_THT:R_Axial_DIN0207_L6.3mm_D2.5mm_P7.62mm_Horizontal, symbol Device:R
- added R28, R29: 1k, Resistor_THT:R_Axial_DIN0207_L6.3mm_D2.5mm_P7.62mm_Horizontal, symbol Device:R
- C5: value 10uF 25V -> 10uF 50V
- TP1, TP2, TP3, TP4, TP5, TP6, TP7, TP8: footprint TestPoint:TestPoint_THTPad_D3.0mm_Drill1.5mm -> fv_reva2:Keystone_5000_Carrier_D3
Connections:
- net +3V3: now also R26.2, R27.2
- net IR_RX1: now also R26.1, R28.2; no longer J9.2 (Pin_2)
- net IR_RX2: now also R27.1, R29.2; no longer J10.2 (Pin_2)
- new net IR_RX1_CABLE: J9.2 (Pin_2), R28.1
- new net IR_RX2_CABLE: J10.2 (Pin_2), R29.1
