File: hardware/FV-CTRL_RevB-02.kicad_sch (KiCad schematic)
At the start: 19 parts, among them U1 ESP32-D0WD-V3

Commit message: feat(hardware): add reset supervisor and thermal EP to bare ESP32 core
Parts:
- added C56: 100nF, Capacitor_SMD:C_0402_1005Metric, symbol Device:C
- added U5: TLV803EA29DBZR, Package_TO_SOT_SMD:SOT-23, symbol fv_revb:TLV803EA29DBZR
Connections:
- net +3V3: now also C56.1, U5.3 (VDD)
- net ESP_EN: now also U5.2 (RESET_OD)
- net GND: now also C56.2, U5.1 (GND)

Commit message: fix(hardware): increase flash brownout margin and account for RF ESD capacitance
Parts:
- U5: value TLV803EA29DBZR -> TLV803EA30DBZR; symbol fv_revb:TLV803EA29DBZR -> fv_revb:TLV803EA30DBZR
Changed lines of the file:
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@@
 	)
 	(symbol
-		(lib_id "fv_revb:TLV803EA29DBZR")
+		(lib_id "fv_revb:TLV803EA30DBZR")
 		(at 259.0800 96.5200 0)
 		(unit 1)
@@
 			(effects (font (size 1.27 1.27)))
 		)
-		(property "Value" "TLV803EA29DBZR"
+		(property "Value" "TLV803EA30DBZR"
 			(at 259.0800 106.6800 0)
 			(effects (font (size 1.27 1.27)))

Commit message: feat(pcb): order QFN escapes and reconnect local supplies before signal routing
Keep two servo rails and GPIO unchanged. Use 0.4/0.2mm escape vias, move C23 to 0201 and preserve ground beneath clock/RF. ERC has zero violations; native DRC has no physical errors or parity differences, with 100 opens and 33 dangling warnings at this intermediate checkpoint. Not a fabrication release.
Parts:
- C23: footprint Capacitor_SMD:C_0402_1005Metric -> Capacitor_SMD:C_0201_0603Metric
Changed lines of the file:
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@@
 			(effects (font (size 1.27 1.27)))
 		)
-		(property "Footprint" "Capacitor_SMD:C_0402_1005Metric"
+		(property "Footprint" "Capacitor_SMD:C_0201_0603Metric"
 			(at 259.0800 180.3400 0)
 			(effects (font (size 1.27 1.27)) (hide yes))
