File: hardware/FV-CTRL_RevB-09.kicad_sch (KiCad schematic)
At the start: 24 parts, among them J21 USB MICRO DATA, Q3 MMBT3904, Q4 MMBT3904, SW1 RESET, SW2 BOOT, U2 CP2102N-A02-GQFN24

Commit message: feat(hardware): add reset supervisor and thermal EP to bare ESP32 core
Parts:
- U2: footprint Package_DFN_QFN:QFN-24-1EP_4x4mm_P0.5mm_EP2.6x2.6mm -> Package_DFN_QFN:QFN-24-1EP_4x4mm_P0.5mm_EP2.6x2.6mm_ThermalVias
Changed lines of the file:
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@@
 			(effects (font (size 1.27 1.27)))
 		)
-		(property "Footprint" "Package_DFN_QFN:QFN-24-1EP_4x4mm_P0.5mm_EP2.6x2.6mm"
+		(property "Footprint" "Package_DFN_QFN:QFN-24-1EP_4x4mm_P0.5mm_EP2.6x2.6mm_ThermalVias"
 			(at 78.7400 106.6800 0)
 			(effects (font (size 1.27 1.27)) (hide yes))

Commit message: feat(pcb): order QFN escapes and reconnect local supplies before signal routing
Keep two servo rails and GPIO unchanged. Use 0.4/0.2mm escape vias, move C23 to 0201 and preserve ground beneath clock/RF. ERC has zero violations; native DRC has no physical errors or parity differences, with 100 opens and 33 dangling warnings at this intermediate checkpoint. Not a fabrication release.
Changed lines of the file:
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@@
 		(dnp no)
 		(property "Reference" "J21"
-			(at 193.0400 38.1000 0)
+			(at 193.0400 26.6400 0)
 			(effects (font (size 1.27 1.27)))
 		)
 		(property "Value" "USB MICRO DATA"
-			(at 193.0400 43.1800 0)
+			(at 193.0400 54.6400 0)
 			(effects (font (size 1.27 1.27)))
 		)
@@
 		(dnp no)
 		(property "Reference" "D9"
-			(at 334.0100 123.1900 0)
+			(at 325.1200 116.4600 0)
 			(effects (font (size 1.27 1.27)))
 		)
 		(property "Value" "PESD5V0X1BL"
-			(at 334.0100 125.7300 0)
+			(at 325.1200 132.4600 0)
 			(effects (font (size 1.27 1.27)))
 		)
@@
 		(dnp no)
 		(property "Reference" "D10"
-			(at 201.9300 151.1300 0)
+			(at 193.0400 144.4000 0)
 			(effects (font (size 1.27 1.27)))
 		)
 		(property "Value" "PESD5V0X1BL"
-			(at 201.9300 153.6700 0)
-			(effects (font (size 1.27 1.27)))
-		)
+			(at 193.0400 160.4000 0)
+			(effects (font (size 1.27 1.27)))
+		)
